File: Oscillator.sch (KiCad schematic (older format))
At the start: 0 parts

Commit message: Added version 1 markings
Other:
- note added: "Oscillator v1"
Changed lines of the file:
@@
 F1 "main.sch" 50
 $EndSheet
+Text Notes 7350 7500 0    50   ~ 0
+Oscillator v1
 $EndSCHEMATC
